Commit message: add some arguments

File: p3dx_description/urdf/pioneer3dx.xacro (robot description, xacro)
@@ -17,4 +17,13 @@
  -->
 <robot name="pioneer3dx" xmlns:xacro="http://ros.org/wiki/xacro">
+  <!--Arguments passed by xacro.py-->
+  <xacro:arg name="contact" default="1"/>
+  <xacro:arg name="laser_noise" default="0.01"/>
+  <xacro:arg name="odom_source" default="world"/>
+  <xacro:arg name="baseFrame" default="base_link"/>
+  <xacro:arg name="mapFrame" default="map"/>
+  <xacro:arg name="worldFrame" default="world"/>
+  <xacro:arg name="odometryFrame" default="odom"/>
+  <xacro:arg name="laserFrame" default="lms100"/>
   <!-- import all gazebo-customization elements, including gazebo colors -->
   <xacro:include filename="$(find p3dx_description)/urdf/pioneer3dx.gazebo" />
@@ -22,204 +31,225 @@
   <xacro:include filename="$(find p3dx_description)/urdf/pioneer3dx_wheel.xacro" />
   <!-- chassis -->
-	<link name="base_link">
-		<inertial>
-			<mass value="3.5" />
-			<!--<origin xyz="-0.025 0 -0.223"/> -->
-			<origin xyz="-0.05 0 0" />
-			<inertia ixx="1" ixy="0" ixz="0" iyy="1" iyz="0" izz="1" />
-		</inertial>
-		<visual name="base_visual">
-			<origin xyz="-0.045 0 0.148" rpy="0 0 0" />
-			<geometry name="pioneer_geom">
-				<mesh filename="package://p3dx_description/meshes/chassis.stl" />
-			</geometry>
-			<material name="ChassisRed">
-				<color rgba="0.851 0.0 0.0 1.0" />
-			</material>
-		</visual>
-		<collision>
-			<origin xyz="-0.045 0 0.145" rpy="0 0 0" />
-			<geometry>
-				<box size="0.35 0.25 0.14" />
-			</geometry>
-		</collision>
-	</link>
+  <link name="base_link">
+    <inertial>
+      <mass value="3.5" />
+      <!--<origin xyz="-0.025 0 -0.223"/> -->
+      <origin xyz="-0.05 0 0" />
+      <inertia ixx="1" ixy="0" ixz="0" iyy="1" iyz="0" izz="1" />
+    </inertial>
+    <visual name="base_visual">
+      <origin xyz="-0.045 0 0.148" rpy="0 0 0" />
+      <geometry name="pioneer_geom">
+        <mesh filename="package://p3dx_description/meshes/chassis.stl" />
+      </geometry>
+      <material name="ChassisRed">
+        <color rgba="0.851 0.0 0.0 1.0" />
+      </material>
+    </visual>
+    <collision name='collision'>
+      <origin xyz="-0.045 0 0.145" rpy="0 0 0" />
+      <geometry>
+        <box size="0.35 0.25 0.14" />
+      </geometry>
+      <surface>
+        <contact collide_without_contact="$(arg contact)" />
+      </surface>
+    </collision>
+  </link>
   <!-- top_plate -->
-	<link name="top_plate">
-		<inertial>
-			<mass value="0.01" />
-			<origin xyz="0 0 0" />
-			<inertia ixx="1" ixy="0" ixz="0" iyy="1" iyz="0" izz="1" />
-		</inertial>
-		<visual name="base_visual">
-			<origin xyz="0 0 0" rpy="0 0 0" />
-			<geometry name="top_geom">
-				<mesh filename="package://p3dx_description/meshes/top.stl" />
-			</geometry>
-			<material name="TopBlack">
-				<color rgba="0.038 0.038 0.038 1.0" />
-			</material>
-		</visual>
-		<collision>
-			<origin xyz="0.0 0 0" rpy="0 0 0" />
-			<geometry name="pioneer_geom">
-				<box size="0.45 0.38 0.01" />
-			</geometry>
-		</collision>
-	</link>
-	<joint name="base_top_joint" type="fixed">
-		<origin xyz="-0.045 0 0.234" rpy="0 0 0" />
-		<parent link="base_link" />
-		<child link="top_plate" />
-	</joint>
+  <link name="top_plate">
+    <inertial>
+      <mass value="0.01" />
+      <origin xyz="0 0 0" />
+      <inertia ixx="1" ixy="0" ixz="0" iyy="1" iyz="0" izz="1" />
+    </inertial>
+    <visual name="base_visual">
+      <origin xyz="0 0 0" rpy="0 0 0" />
+      <geometry name="top_geom">
+        <mesh filename="package://p3dx_description/meshes/top.stl" />
+      </geometry>
+      <material name="TopBlack">
+        <color rgba="0.038 0.038 0.038 1.0" />
+      </material>
+    </visual>
+    <collision name='collision'>
+      <origin xyz="0.0 0 0" rpy="0 0 0" />
+      <geometry name="pioneer_geom">
+        <box size="0.45 0.38 0.01" />
+      </geometry>
+      <surface>
+        <contact collide_without_contact="$(arg contact)" />
+      </surface>
+    </collision>
+  </link>
+  <joint name="base_top_joint" type="fixed">
+    <origin xyz="-0.045 0 0.234" rpy="0 0 0" />
+    <parent link="base_link" />
+    <child link="top_plate" />
+  </joint>
   <!-- swivel -->
-	<link name="swivel">
-		<inertial>
-			<mass value="0.1" />
-			<origin xyz="0 0 0" />
-			<inertia ixx="0.01" ixy="0" ixz="0" iyy="0.01" iyz="0" izz="0.01" />
-		</inertial>
-		<visual name="base_visual">
-			<origin xyz="0 0 0" rpy="0 0 0" />
-			<geometry name="pioneer_geom">
-				<mesh filename="package://p3dx_description/meshes/swivel.stl" />
-			</geometry>
-			<material name="swivel">
-				<color rgba="0.5 0.5 0.5 1" />
-			</material>
-		</visual>
-		<collision>
-			<origin xyz="0 0 0" rpy="0 0 0" />
-			<geometry>
-				<box size="0 0 0" />
-			</geometry>
-		</collision>
-	</link>
-	<joint name="base_swivel_joint" type="continuous">
-		<origin xyz="-0.185 0 0.055" rpy="0 0 0" />
-		<axis xyz="0 0 1" />
-		<anchor xyz="0 0 0" />
-		<limit effort="100" velocity="100" k_velocity="0" />
-		<joint_properties damping="0.0" friction="0.0" />
-		<parent link="base_link" />
-		<child link="swivel" />
-	</joint>
+  <link name="swivel">
+    <inertial>
+      <mass value="0.1" />
+      <origin xyz="0 0 0" />
+      <inertia ixx="0.01" ixy="0" ixz="0" iyy="0.01" iyz="0" izz="0.01" />
+    </inertial>
+    <visual name="base_visual">
+      <origin xyz="0 0 0" rpy="0 0 0" />
+      <geometry name="pioneer_geom">
+        <mesh filename="package://p3dx_description/meshes/swivel.stl" />
+      </geometry>
+      <material name="swivel">
+        <color rgba="0.5 0.5 0.5 1" />
+      </material>
+    </visual>
+    <collision name='collision'>
+      <origin xyz="0 0 0" rpy="0 0 0" />
+      <geometry>
+        <box size="0 0 0" />
+      </geometry>
+      <surface>
+        <contact collide_without_contact="$(arg contact)" />
+      </surface>
+    </collision>
+  </link>
+  <joint name="base_swivel_joint" type="continuous">
+    <origin xyz="-0.185 0 0.055" rpy="0 0 0" />
+    <axis xyz="0 0 1" />
+    <anchor xyz="0 0 0" />
+    <limit effort="100" velocity="100" k_velocity="0" />
+    <joint_properties damping="0.0" friction="0.0" />
+    <parent link="base_link" />
+    <child link="swivel" />
+  </joint>
   <!-- center_hubcap -->
-	<link name="center_hubcap">
-		<inertial>
-			<mass value="0.01" />
-			<origin xyz="0 0 0" />
-			<inertia ixx="0.012411765597" ixy="-0.000711733678" ixz="0.00050272983"
-				iyy="0.015218160428" iyz="-0.000004273467" izz="0.011763977943" />
-		</inertial>
-		<visual name="base_visual">
-			<origin xyz="0 0 0" rpy="0 0 0" />
-			<geometry name="pioneer_geom">
-				<mesh filename="package://p3dx_description/meshes/center_hubcap.stl" />
-			</geometry>
-			<material name="swivel">
-				<color rgba="0.5 0.5 0.5 1" />
-			</material>
-		</visual>
-		<collision>
-			<origin xyz="0 0 0" rpy="0 0 0" />
-			<geometry>
-				<box size="0 0 0" />
-			</geometry>
-		</collision>
-	</link>
-	<joint name="swivel_hubcap_joint" type="continuous">
-		<origin xyz="-0.026 0 -0.016" rpy="0 0 0" />
-		<axis xyz="0 1 0" />
-		<anchor xyz="0 0 0" />
-		<limit effort="100" velocity="100" k_velocity="0" />
-		<joint_properties damping="0.0" friction="0.0" />
-		<parent link="swivel" />
-		<child link="center_wheel" />
-	</joint>
+  <link name="center_hubcap">
+    <inertial>
+      <mass value="0.01" />
+      <origin xyz="0 0 0" />
+      <inertia ixx="0.012411765597" ixy="-0.000711733678" ixz="0.00050272983"
+        iyy="0.015218160428" iyz="-0.000004273467" izz="0.011763977943" />
+    </inertial>
+    <visual name="base_visual">
+      <origin xyz="0 0 0" rpy="0 0 0" />
+      <geometry name="pioneer_geom">
+        <mesh filename="package://p3dx_description/meshes/center_hubcap.stl" />
+      </geometry>
+      <material name="swivel">
+        <color rgba="0.5 0.5 0.5 1" />
+      </material>
+    </visual>
+    <collision name='collision'>
+      <origin xyz="0 0 0" rpy="0 0 0" />
+      <geometry>
+        <box size="0 0 0" />
+      </geometry>
+      <surface>
+        <contact collide_without_contact="$(arg contact)" />
+      </surface>
+    </collision>
+  </link>
+  <joint name="swivel_hubcap_joint" type="continuous">
+    <origin xyz="-0.026 0 -0.016" rpy="0 0 0" />
+    <axis xyz="0 1 0" />
+    <anchor xyz="0 0 0" />
+    <limit effort="100" velocity="100" k_velocity="0" />
+    <joint_properties damping="0.0" friction="0.0" />
+    <parent link="swivel" />
+    <child link="center_wheel" />
+  </joint>
   <!-- center_wheel -->
-	<link name="center_wheel">
-		<inertial>
-			<mass value="0.1" />
-			<origin xyz="0 0 0" />
-			<inertia ixx="0.012411765597" ixy="-0.000711733678" ixz="0.00050272983"
-				iyy="0.015218160428" iyz="-0.000004273467" izz="0.011763977943" />
-		</inertial>
-		<visual name="base_visual">
-			<origin xyz="0 0 0" rpy="0 0 0" />
-			<geometry name="pioneer_geom">
-				<mesh filename="package://p3dx_description/meshes/center_wheel.stl" />
-			</geometry>
-			<material name="WheelBlack">
-				<color rgba="0.117 0.117 0.117 1" />
-			</material>
-		</visual>
-		<collision>
-			<origin xyz="0 0 0" rpy="${-3.1415927/2.0} 0 0" />
-			<geometry>
-				<cylinder radius="0.0375" length="0.01" />
-			</geometry>
-		</collision>
-	</link>
-	<joint name="center_wheel_joint" type="fixed">
-		<origin xyz="-0.0035 0 -0.001" rpy="0 0 0"/>
-		<parent link="center_wheel"/>
-		<child link="center_hubcap"/>
-	</joint>
-	<xacro:p3dx_wheel suffix="left" parent="base_link" reflect="1"/>
-	<xacro:p3dx_wheel suffix="right" parent="base_link" reflect="-1"/>
+  <link name="center_wheel">
+    <inertial>
+      <mass value="0.1" />
+      <origin xyz="0 0 0" />
+      <inertia ixx="0.012411765597" ixy="-0.000711733678" ixz="0.00050272983"
+        iyy="0.015218160428" iyz="-0.000004273467" izz="0.011763977943" />
+    </inertial>
+    <visual name="base_visual">
+      <origin xyz="0 0 0" rpy="0 0 0" />
+      <geometry name="pioneer_geom">
+        <mesh filename="package://p3dx_description/meshes/center_wheel.stl" />
+      </geometry>
+      <material name="WheelBlack">
+        <color rgba="0.117 0.117 0.117 1" />
+      </material>
+    </visual>
+    <collision name='collision'>
+      <origin xyz="0 0 0" rpy="${-3.1415927/2.0} 0 0" />
+      <geometry>
+        <cylinder radius="0.0375" length="0.01" />
+      </geometry>
+      <surface>
+        <contact collide_without_contact="$(arg contact)" />
+      </surface>
+    </collision>
+  </link>
+  <joint name="center_wheel_joint" type="fixed">
+    <origin xyz="-0.0035 0 -0.001" rpy="0 0 0"/>
+    <parent link="center_wheel"/>
+    <child link="center_hubcap"/>
+  </joint>
+  <xacro:p3dx_wheel suffix="left" parent="base_link" reflect="1" contact="$(arg contact)"/>
+  <xacro:p3dx_wheel suffix="right" parent="base_link" reflect="-1" contact="$(arg contact)"/>
   <!-- front_sonar -->
-	<link name="front_sonar">
-		<inertial>
-			<mass value="0.0001" />
-			<origin xyz="0 0 0" />
-			<inertia ixx="1" ixy="0" ixz="0" iyy="1" iyz="0" izz="1" />
-		</inertial>
-		<visual name="front_sonar_vis">
-			<origin rpy="0 0 0" xyz="0 0 0" />
-			<geometry name="pioneer_geom">
-				<mesh filename="package://p3dx_description/meshes/front_sonar.stl" />
-			</geometry>
-			<material name="SonarYellow">
-				<color rgba="0.715 0.583 0.210 1.0" />
-			</material>
-		</visual>
-		<collision>
-			<origin rpy="0 0 0" xyz="0 0 0" />
-			<geometry>
-				<box size="0 0 0" />
-			</geometry>
-		</collision>
-	</link>
-	<joint name="base_front_joint" type="fixed">
-		<origin rpy="0 0 0" xyz="0.109 0 0.209" />
-		<parent link="base_link" />
-		<child link="front_sonar" />
-	</joint>
-	<!-- lms100 laser -->
-	<link name="lms100">
-		<inertial>
-			<mass value="1e-5" />
-			<origin xyz="0 0 0" rpy="0 0 0" />
-			<inertia ixx="1e-6" ixy="0" ixz="0" iyy="1e-6" iyz="0" izz="1e-6" />
-		</inertial>
-		<visual>
-			<origin xyz="0 0 0" rpy="0 0 0" />
-			<geometry>
-				<mesh filename="package://p3dx_description/meshes/lms100.dae" />
-			</geometry>
-		</visual>
-		<collision>
-			<origin xyz="0 0 0" rpy="0 0 0" />
-			<geometry>
-				<box size="0.1 0.1 0.1" />
-			</geometry>
-		</collision>
-	</link>
-	<joint name="lms100_joint" type="fixed">
-		<axis xyz="0 1 0" />
-		<origin xyz="0.16 0 0.15" rpy="0 0 0" />
-		<parent link="base_link" />
-		<child link="lms100" />
-	</joint>
+  <link name="front_sonar">
+    <inertial>
+      <mass value="0.0001" />
+      <origin xyz="0 0 0" />
+      <inertia ixx="1" ixy="0" ixz="0" iyy="1" iyz="0" izz="1" />
+    </inertial>
+    <visual name="front_sonar_vis">
+      <origin rpy="0 0 0" xyz="0 0 0" />
+      <geometry name="pioneer_geom">
+        <mesh filename="package://p3dx_description/meshes/front_sonar.stl" />
+      </geometry>
+      <material name="SonarYellow">
+        <color rgba="0.715 0.583 0.210 1.0" />
+      </material>
+    </visual>
+    <collision name='collision'>
+      <origin rpy="0 0 0" xyz="0 0 0" />
+      <geometry>
+        <box size="0 0 0" />
+      </geometry>
+      <surface>
+        <contact collide_without_contact="$(arg contact)" />
+      </surface>
+    </collision>
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
File: p3dx_description/urdf/pioneer3dx_wheel.xacro (robot description, xacro)
@@ -17,92 +17,102 @@
  -->
 <robot xmlns:xacro="http://ros.org/wiki/xacro">
-	<!-- properties (constants) -->
-	<property name="M_PI" value="3.14159" />
-	<!-- right/left hubcap + wheel -->
-	<xacro:macro name="p3dx_wheel" params="suffix parent reflect">
-		<!-- wheel -->
-		<link name="p3dx_${suffix}_wheel">
-			<inertial>
-				<mass value="0.5" />
-				<origin xyz="0 0 0" />
-				<inertia ixx="0.012411765597" ixy="0" ixz="0" iyy="0.015218160428"
-					iyz="0" izz="0.011763977943" />
-			</inertial>
-			<visual name="base_visual">
-				<origin xyz="0 0 0" rpy="0 0 0" />
-				<geometry name="pioneer_geom">
-					<mesh filename="package://p3dx_description/meshes/${suffix}_wheel.stl" />
-				</geometry>
-				<material name="WheelBlack">
-					<color rgba="0.117 0.117 0.117 1" />
-				</material>
-			</visual>
-			<collision>
-				<origin xyz="0 0 0" rpy="${-3.1415927/2} 0 0" />
-				<geometry>
-					<!--<mesh filename="package://p3dx_description/meshes/${suffix}_wheel.stl"/> -->
-					<cylinder radius="0.09" length="0.01" />
-				</geometry>
-			</collision>
-		</link>
-		<joint name="base_${suffix}_hubcap_joint" type="fixed">
-			<origin xyz="0 0 0" rpy="0 0 0" />
-			<parent link="p3dx_${suffix}_wheel" />
-			<child link="p3dx_${suffix}_hubcap" />
-		</joint>
-		<!-- hubcap -->
-		<link name="p3dx_${suffix}_hubcap">
-			<inertial>
-				<mass value="0.01" />
-				<origin xyz="0 0 0" />
-				<inertia ixx="0.012411765597" ixy="0" ixz="0" iyy="0.015218160428"
-					iyz="0" izz="0.011763977943" />
-			</inertial>
-			<visual name="base_visual">
-				<origin xyz="0 0 0" rpy="0 0 0" />
-				<geometry name="pioneer_geom">
-					<mesh filename="package://p3dx_description/meshes/${suffix}_hubcap.stl" />
-				</geometry>
-				<material name="HubcapYellow">
-					<color rgba="1.0 0.811 0.151 1.0" />
-				</material>
-			</visual>
-			<collision>
-				<origin xyz="0 0 0" rpy="0 0 0" />
-				<geometry>
-					<box size="0 0 0" />
-				</geometry>
-			</collision>
-		</link>
-		<joint name="base_${suffix}_wheel_joint" type="continuous">
-			<axis xyz="0 1 0" />
-			<anchor xyz="0 0 0" />
-			<limit effort="100" velocity="100" />
-			<joint_properties damping="0.0" friction="0.0" />
-			<origin xyz="0 ${reflect*0.158} 0.091" rpy="0 0 0" />
-			<parent link="base_link" />
-			<child link="p3dx_${suffix}_wheel" />
-		</joint>
-		<!-- gazebo elements -->
-		<transmission name="${parent}_${suffix}_wheel_trans">
-			<type>transmission_interface/SimpleTransmission</type>
-			<joint name="base_${suffix}_wheel_joint">
-				<hardwareInterface>EffortJointInterface</hardwareInterface>
-			</joint>
-			<actuator name="base_${suffix}_wheel_motor">
-				<hardwareInterface>EffortJointInterface</hardwareInterface>
-				<mechanicalReduction>${reflect * 624/35 * 80/19}</mechanicalReduction>
-			</actuator>
-		</transmission>
-		<gazebo reference="p3dx_${suffix}_hubcap">
-			<material>Gazebo/Yellow</material>
-		</gazebo>
-		<gazebo reference="p3dx_${suffix}_wheel">
-			<material>Gazebo/Black</material>
-			<mu1>0.5</mu1>
-			<mu2>50.0</mu2>
-			<kp>100000000.0</kp>
-			<kd>1.0</kd>
-		</gazebo>
-	</xacro:macro>
+  <!-- properties (constants) -->
+  <property name="M_PI" value="3.14159" />
+  <!-- right/left hubcap + wheel -->
+  <xacro:macro name="p3dx_wheel" params="suffix parent reflect contact">
+    <!-- link wheel -->
+    <link name="p3dx_${suffix}_wheel">
+      <inertial>
+        <mass value="0.5" />
+        <origin xyz="0 0 0" />
+        <inertia ixx="0.012411765597" ixy="0" ixz="0" iyy="0.015218160428"
+          iyz="0" izz="0.011763977943" />
+      </inertial>
+      <visual name="base_visual">
+        <origin xyz="0 0 0" rpy="0 0 0" />
+        <geometry name="pioneer_geom">
+          <mesh filename="package://p3dx_description/meshes/${suffix}_wheel.stl" />
+        </geometry>
+        <material name="WheelBlack">
+          <color rgba="0.117 0.117 0.117 1" />
+        </material>
+      </visual>
+      <collision name='collision'>
+        <origin xyz="0 0 0" rpy="${-3.1415927/2} 0 0" />
+        <geometry>
+          <!--<mesh filename="package://p3dx_description/meshes/${suffix}_wheel.stl"/> -->
+          <cylinder radius="0.09" length="0.01" />
+        </geometry>
+        <surface>
+          <contact collide_without_contact="${contact}"/>
+        </surface>
+      </collision>
+    </link>
+    <!-- joint wheel to hubcap-->
+    <joint name="base_${suffix}_hubcap_joint" type="fixed">
+      <origin xyz="0 0 0" rpy="0 0 0" />
+      <parent link="p3dx_${suffix}_wheel" />
+      <child link="p3dx_${suffix}_hubcap" />
+    </joint>
+    <!-- link hubcap -->
+    <link name="p3dx_${suffix}_hubcap">
+      <inertial>
+        <mass value="0.01" />
+        <origin xyz="0 0 0" />
+        <inertia ixx="0.012411765597" ixy="0" ixz="0" iyy="0.015218160428"
+          iyz="0" izz="0.011763977943" />
+      </inertial>
+      <visual name="base_visual">
+        <origin xyz="0 0 0" rpy="0 0 0" />
+        <geometry name="pioneer_geom">
+          <mesh filename="package://p3dx_description/meshes/${suffix}_hubcap.stl" />
+        </geometry>
+        <material name="HubcapYellow">
+          <color rgba="1.0 0.811 0.151 1.0" />
+        </material>
+      </visual>
+      <collision name='collision'>
+        <origin xyz="0 0 0" rpy="0 0 0" />
+        <geometry>
+          <box size="0 0 0" />
+        </geometry>
+        <surface>
+          <contact collide_without_contact="${contact}"/>
+        </surface>
+      </collision>
+    </link>
+    <!-- joint ${parent} to wheel -->
+    <joint name="base_${suffix}_wheel_joint" type="continuous">
+      <axis xyz="0 1 0" />
+      <anchor xyz="0 0 0" />
+      <limit effort="100" velocity="100" />
+      <joint_properties damping="0.0" friction="0.0" />
+      <origin xyz="0 ${reflect*0.158} 0.091" rpy="0 0 0" />
+      <parent link="${parent}" />
+      <child link="p3dx_${suffix}_wheel" />
+    </joint>
+    <!-- gazebo wheel_joint -->
+    <transmission name="${parent}_${suffix}_wheel_trans">
+      <type>transmission_interface/SimpleTransmission</type>
+      <joint name="base_${suffix}_wheel_joint">
+        <hardwareInterface>EffortJointInterface</hardwareInterface>
+      </joint>
+      <actuator name="base_${suffix}_wheel_motor">
+        <hardwareInterface>EffortJointInterface</hardwareInterface>
+        <mechanicalReduction>${reflect * 624/35 * 80/19}</mechanicalReduction>
+      </actuator>
+    </transmission>
+    <!-- gazebo hubcap -->
+    <gazebo reference="p3dx_${suffix}_hubcap">
+      <material>Gazebo/Yellow</material>
+    </gazebo>
+    <!-- gazego wheel -->
+    <gazebo reference="p3dx_${suffix}_wheel">
+      <material>Gazebo/Black</material>
+      <mu1>0.5</mu1><!--friction coefficient-->
+      <mu2>50.0</mu2>
+      <kp>100000000.0</kp><!--stiffness-->
+      <kd>1.0</kd><!--damping-->
+    </gazebo>
+  </xacro:macro>
 </robot>

Commit message: move joint_state_publishers from p3dx_2dnav to p3dx_gazebo

File: p3dx_description/urdf/pioneer3dx.xacro (robot description, xacro)
@@ -21,9 +21,9 @@
   <xacro:arg name="laser_noise" default="0.01"/>
   <xacro:arg name="odom_source" default="world"/>
-  <xacro:arg name="baseFrame" default="base_link"/>
-  <xacro:arg name="mapFrame" default="map"/>
-  <xacro:arg name="worldFrame" default="world"/>
-  <xacro:arg name="odometryFrame" default="odom"/>
-  <xacro:arg name="laserFrame" default="lms100"/>
+  <xacro:arg name="base_frame" default="base_link"/>
+  <xacro:arg name="map_frame" default="map"/>
+  <xacro:arg name="world_frame" default="world"/>
+  <xacro:arg name="odometry_frame" default="odom"/>
+  <xacro:arg name="laser_frame" default="lms100"/>
   <!-- import all gazebo-customization elements, including gazebo colors -->
   <xacro:include filename="$(find p3dx_description)/urdf/pioneer3dx.gazebo" />
@@ -225,5 +225,5 @@
   </joint>
   <!-- lms100 laser -->
-  <link name="$(arg laserFrame)">
+  <link name="$(arg laser_frame)">
     <inertial>
       <mass value="1e-5" />
@@ -247,9 +247,9 @@
     </collision>
   </link>
-  <joint name="base_$(arg laserFrame)_joint" type="fixed">
+  <joint name="base_$(arg laser_frame)_joint" type="fixed">
     <axis xyz="0 1 0" />
     <origin xyz="0.16 0 0.15" rpy="0 0 0" />
     <parent link="base_link" />
-    <child link="$(arg laserFrame)" />
+    <child link="$(arg laser_frame)" />
   </joint>
 </robot>
